File: Hardware/SparkFun GPS RTK Surveyor.brd (EAGLE design)
At the start: 68.2 x 110.1 mm, 197 parts, among them J13 Internal, J16 microSD, J17 Qwiic Right Angle, J3 USB Female Type C Connector, J4 External, J5 USB Female Type C Connector, J6 Start Base, J7 Power Switch, Q2 MBT3904DW1T1, U1 ESP-WROOM-3232D-NARROW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

Commit message: Replace SMA SMD with edge mount SMA. v17 PCB
Parts:
- added U$94, U$95: (no value), output:V170
- E1: device SparkFun-RF:SMA-EDGE-SMD -> SparkFun-RF:SMA-EDGE
- moved E1 3.54 mm to (14.0, 3.66)
Connections:
- net GND: now also E1.GND@2, E1.GND@3
Routing:
- net GPS_ANT1: track 14.2 -> 18.8 mm
- net GND: vias 194 -> 189
Other:
- outline, holes or cut-outs redrawn
- board text removed: "v16"
Changed lines of the file:
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@@
 <setting verticaltext="up"/>
 </settings>
-<grid distance="0.05" unitdist="inch" unit="inch" style="lines" multiple="1" display="yes" altdistance="0.005" altunitdist="inch" altunit="inch"/>
+<grid distance="1" unitdist="mm" unit="mm" style="lines" multiple="1" display="yes" altdistance="0.1" altunitdist="mm" altunit="mm"/>
 <layers>
 <layer number="1" name="Top" color="4" fill="1" visible="yes" active="yes"/>
@@
 <board>
 <plain>
-<text x="2.794" y="108.839" size="1.27" layer="1" font="vector" ratio="15" rot="SR0" align="center">v16</text>
 <text x="74.93" y="63.5" size="1.778" layer="51" font="vector" ratio="15">No clean process</text>
 <text x="74.93" y="66.04" size="1.778" layer="51" font="vector" ratio="15">4 Layer Board</text>
@@
 <wire x1="-3.175" y1="50.165" x2="-3.175" y2="56.515" width="0.2032" layer="20" curve="180"/>
 <wire x1="53.975" y1="50.165" x2="53.975" y2="56.515" width="0.2032" layer="20" curve="-180"/>
-<wire x1="-3.6" y1="0.065" x2="54.4" y2="0.065" width="0.2032" layer="20"/>
+<wire x1="-3.6" y1="0.065" x2="9.748" y2="0.065" width="0.2032" layer="20"/>
+<wire x1="18.248" y1="0.065" x2="54.4" y2="0.065" width="0.2032" layer="20"/>
 <wire x1="-3.6" y1="0.065" x2="-3.6" y2="3.34" width="0.2032" layer="20"/>
 <wire x1="-3.6" y1="3.34" x2="-5.35" y2="3.34" width="0.2032" layer="20"/>
@@
 <wire x1="59.436" y1="76.2" x2="58.928" y2="85.09" width="0.2032" layer="20"/>
 <text x="74.93" y="68.58" size="1.778" layer="51" font="vector" ratio="15">Board thickness is 1.6mm</text>
+<wire x1="18.248" y1="0.065" x2="18.248" y2="1.381" width="0.2032" layer="20"/>
+<wire x1="18.248" y1="1.381" x2="9.748" y2="1.381" width="0.2032" layer="20"/>
+<wire x1="9.748" y1="1.381" x2="9.748" y2="0.065" width="0.2032" layer="20"/>
 </plain>
 <attributes>
@@
 <attribute name="VALUE" x="25.03" y="13.97" size="0.6096" layer="27" ratio="20" rot="R90" align="top-center"/>
 </element>
-<element name="E1" library="SparkFun-RF" package="SMA-EDGE-SMD" value="SMA" x="13.97" y="0.111" smashed="yes" rot="R180">
-<attribute name="PROD_ID" value="CONN-15100" x="13.97" y="0.111" size="1.778" layer="27" rot="R180" display="off"/>
+<element name="E1" library="SparkFun-RF" package="SMA-EDGE" value="SMA" x="13.97" y="3.656" smashed="yes" rot="R180">
+<attribute name="PROD_ID" value="CONN-08289" x="13.97" y="3.656" size="1.778" layer="27" rot="R180" display="off"/>
 </element>
 <element name="U$30" library="SparkFun-Aesthetics" package="QWIIC_4MM" value="" x="25.4" y="6.715" smashed="yes" rot="MR0"/>
@@
 <attribute name="VALUE" x="25.4" y="87.44" size="0.8128" layer="28" rot="MR180" align="center"/>
 </element>
+<element name="U$94" library="output" package="V170" value="" x="38.1" y="99.06" smashed="yes"/>
+<element name="U$95" library="output" package="V170" value="" x="25.4" y="48.26" smashed="yes" rot="MR0"/>
 </elements>
 <signals>
@@
 <via x="15.24" y="12.022" extent="1-16" drill="0.3048"/>
 <via x="12.954" y="8.144" extent="1-16" drill="0.3048"/>
-<via x="11.938" y="8.62" extent="1-16" drill="0.3048"/>
-<via x="16.51" y="8.747" extent="1-16" drill="0.3048"/>
-<via x="10.541" y="8.493" extent="1-16" drill="0.3048"/>
-<via x="8.763" y="7.89" extent="1-16" drill="0.3048"/>
+<via x="12.338" y="6.92" extent="1-16" drill="0.3048"/>
+<via x="16.41" y="6.747" extent="1-16" drill="0.3048"/>
 <via x="15.113" y="7.89" extent="1-16" drill="0.3048"/>
-<via x="8.509" y="6.493" extent="1-16" drill="0.3048"/>
-<via x="8.509" y="5.096" extent="1-16" drill="0.3048"/>
-<via x="8.509" y="3.699" extent="1-16" drill="0.3048"/>
+<via x="10.909" y="6.693" extent="1-16" drill="0.3048"/>
+<via x="9.709" y="5.696" extent="1-16" drill="0.3048"/>
+<via x="9.709" y="3.999" extent="1-16" drill="0.3048"/>
 <via x="8.509" y="0.905" extent="1-16" drill="0.3048"/>
-<via x="8.509" y="2.302" extent="1-16" drill="0.3048"/>
+<via x="9.709" y="2.402" extent="1-16" drill="0.3048"/>
 <via x="16.256" y="12.684" extent="1-16" drill="0.3048"/>
 <via x="17.145" y="13.2" extent="1-16" drill="0.3048"/>
@@
 <via x="19.812" y="15.367" extent="1-16" drill="0.3048"/>
 <via x="17.961" y="12.022" extent="1-16" drill="0.3048"/>
-<via x="18.034" y="7.89" extent="1-16" drill="0.3048"/>
-<via x="19.431" y="7.763" extent="1-16" drill="0.3048"/>
-<via x="19.304" y="6.493" extent="1-16" drill="0.3048"/>
-<via x="19.304" y="4.969" extent="1-16" drill="0.3048"/>
-<via x="19.304" y="3.826" extent="1-16" drill="0.3048"/>
-<via x="19.304" y="2.302" extent="1-16" drill="0.3048"/>
+<via x="18.304" y="6.069" extent="1-16" drill="0.3048"/>
+<via x="18.304" y="4.326" extent="1-16" drill="0.3048"/>
+<via x="18.304" y="2.802" extent="1-16" drill="0.3048"/>
 <via x="19.304" y="0.905" extent="1-16" drill="0.3048"/>
 <via x="20.447" y="17.907" extent="1-16" drill="0.3048"/>
@@
 <contactref element="U1" pad="GND1"/>
 <contactref element="U1" pad="GNDT8"/>
+<contactref element="E1" pad="GND@2"/>
+<contactref element="E1" pad="GND@3"/>
 </signal>
 <signal name="ESP_22/SCL">
@@
 <wire x1="19.35" y1="19.22" x2="19.35" y2="18.048" width="0.35051875" layer="1"/>
 <wire x1="13.97" y1="12.668" x2="13.97" y2="10.8" width="0.35051875" layer="1"/>
-<wire x1="13.97" y1="10.8" x2="13.97" y2="8.211" width="0.35051875" layer="1"/>
+<wire x1="13.97" y1="10.8" x2="13.97" y2="3.656" width="0.35051875" layer="1"/>
 <wire x1="13.97" y1="12.68583125" x2="13.97" y2="12.668" width="0.35" layer="1"/>
 <wire x1="19.439" y1="16.891" x2="18.17516875" y2="16.891" width="0.35" layer="1"/>
